File: Carte_arriere_acquisition.kicad_pcb (KiCad board)
At the start: 2 copper layers, 15 parts, among them J1 Screw_Terminal_01x02, J2 Vers_BMS, J3 Vers_Thermistor, J4 Vers_Capteur_Hall, J5 Conn_01x04_Pin, J6 Conn_01x04_Pin, U1 ESP32-DEVKITC-32E, U2 SN65HVD230, U3 MAX3485

Commit message: Modif PCB
Parts:
- removed C1, C2, C3: 100nF, Capacitor_SMD:C_0805_2012Metric_Pad1.18x1.45mm_HandSolder
- removed J1: Screw_Terminal_01x02, TerminalBlock_Phoenix:TerminalBlock_Phoenix_MKDS-1,5-2_1x02_P5.00mm_Horizontal
- removed J2: Vers_BMS, TerminalBlock_Phoenix:TerminalBlock_Phoenix_MKDS-1,5-2_1x02_P5.00mm_Horizontal
- removed J3: Vers_Thermistor, TerminalBlock_Phoenix:TerminalBlock_Phoenix_MKDS-1,5-2_1x02_P5.00mm_Horizontal
- removed J4: Vers_Capteur_Hall, TerminalBlock_Phoenix:TerminalBlock_Phoenix_MKDS-1,5-3_1x03_P5.00mm_Horizontal
- removed J5, J6: Conn_01x04_Pin, Connector_PinHeader_1.27mm:PinHeader_1x04_P1.27mm_Vertical
- removed R1: 1k, Resistor_SMD:R_0805_2012Metric_Pad1.20x1.40mm_HandSolder
- removed R2: 120, Resistor_SMD:R_0805_2012Metric_Pad1.20x1.40mm_HandSolder
- removed R3: 10k, Resistor_SMD:R_0805_2012Metric_Pad1.20x1.40mm_HandSolder
- removed U1: ESP32-DEVKITC-32E, ESP32-DEVKITC-32E:MODULE_ESP32-DEVKITC-32E
- removed U2: SN65HVD230, Package_SO:SOIC-8_3.9x4.9mm_P1.27mm
- removed U3: MAX3485, Package_SO:SOIC-8_3.9x4.9mm_P1.27mm
Routing:
- net Net-(J1-Pin_2): track 15.9 -> 0.00 mm
- net /BMS TX: track 14.3 -> 0.00 mm
- net /BMS_Direction: track 13.4 -> 0.00 mm
- net Net-(J2-Pin_2): track 12.6 -> 0.00 mm
- net Net-(J1-Pin_1): track 12.1 -> 0.00 mm
- net /BMS RX: track 8.84 -> 0.00 mm
- net /Hall: track 8.29 -> 0.00 mm
- net Net-(J2-Pin_1): track 7.04 -> 0.00 mm
- net GND: track 2.68 -> 0.00 mm
